File: eagle/AD8402_WeinBridge_DCO/AD8402_WeinBridge_DCO.sch (EAGLE design)
At the start: 22 parts, among them IC1 NJM2732, IC2 AD8402_DIP14, IC3 TLE2426LP

Commit message: Before Routing Board Design
Parts:
- added JP4: TP_GND, pinhead:PINHD-1X2
- added JP5: SPI, pinhead:PINHD-1X4
- added JP6: OUT, pinhead:PINHD-1X2
- added JP7: PWR, pinhead:PINHD-1X2
- added LED1: GREEN, led:LED3MM
- added R6: 1k, rcl:R-EU_0207/7
- C3: value 10uF -> 100uF; device rcl:CPOL-EUE2.5-5 -> rcl:CPOL-EUE2.5-7
Connections:
- new net N$7: LED1.A, R6.1
- net +5V: now also JP7.1, R6.2
- net CS: now also JP5.3
- net GND: now also JP4.1, JP4.2, JP5.4, JP6.2, JP7.2, LED1.C
- net MOSI: now also JP5.2
- net N$1: now also R2.2; no longer R1.E, R1.S
- net N$2: now also R1.E, R2.1; no longer R1.A, R2.2
- net N$4: now also JP6.1
- net SCK: now also JP5.1
- net VCC/2: now also R1.A, R1.S; no longer R2.1
Other:
- moved on the sheet: C5, C6, C7, C8, C9, IC3, JP3, R1, R2

Commit message: Update eagle files
Connections:
- removed net N$7: LED1.A, R6.1
- new net N$3: LED1.C, R6.2
- net +5V: now also LED1.A; no longer R6.2
- net GND: now also R6.1; no longer LED1.C
Other:
- note added: "※C1、C2は特性を揃える"
- moved on the sheet: C1, C2, C3, C4, C5, C6, C7, C8, C9, D1, D2, IC1A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
